Commit message: Changed robot look properties

File: Project2/my_robot/urdf/my_robot.xacro (robot description, xacro)
@@ -175,5 +175,5 @@
 <!-- robot colours -->
   <gazebo reference="left_wheel">
-    <material>Gazebo/Green</material>
+    <material>Gazebo/Red</material>
   </gazebo>
   <gazebo reference="right_wheel">
@@ -181,8 +181,11 @@
   </gazebo>
   <gazebo reference="chassis">
+    <material>Gazebo/DarkGrey</material>
+  </gazebo>
+  <gazebo reference="camera">
     <material>Gazebo/Blue</material>
   </gazebo>
-  <gazebo reference="camera">
-    <material>Gazebo/Red</material>
+  <gazebo reference="hokuyo">
+    <material>Gazebo/YellowGlow</material>
   </gazebo>
 </robot>
