Commit message: before mapping

File: Project4/my_robot/urdf/my_robot.xacro (robot description, xacro)
@@ -145,4 +145,12 @@
     <parent link="chassis"/>
   </joint>
+  <!-- RGB-D camera -->
+  <joint name="camera_optical_joint" type="fixed">
+    <origin xyz="0 0 0" rpy="-1.5707 0 -1.5707"/>
+    <parent link="camera"/>
+    <child link="camera_link_optical"/>
+  </joint>
+  <link name="camera_link_optical">
+  </link>
 <!-- hokuyo lidar sensor -->
   <link name="hokuyo">
